File: RN171ZigBeeFootprintPCB_RV1/RN-XV_ZigBeeFootprint.sch (EAGLE design)
At the start: 4 parts

Commit message: Connecting GND to the circuit
Changed lines of the file:
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@@
 <?xml version="1.0" encoding="utf-8"?>
 <!DOCTYPE eagle SYSTEM "eagle.dtd">
-<eagle version="6.6.0">
+<eagle version="6.1">
 <drawing>
 <settings>
@@
 <part name="J2" library="con-amp" deviceset="MTA08-100" device=""/>
 <part name="J3" library="con-amp" deviceset="MTA08-100" device=""/>
-<part name="U$1" library="eka_logo" deviceset="EKA_LOGO" device=""/>
 </parts>
 <sheets>
@@
 <instance part="J2" gate="G$1" x="107.95" y="125.73" rot="MR270"/>
 <instance part="J3" gate="G$1" x="210.82" y="95.25" rot="R270"/>
-<instance part="U$1" gate="G$1" x="60.96" y="73.66"/>
 </instances>
 <busses>

Commit message: Connecting RN171's 34 pin to VCC
Connections:
- removed net VCC: XB1.VCC
- net VDD_3.3V: now also J1.VDD_3.3V_RF, J1.VDD_BATT, XB1.VCC
Changed lines of the file:
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@@
 <?xml version="1.0" encoding="utf-8"?>
 <!DOCTYPE eagle SYSTEM "eagle.dtd">
-<eagle version="6.1">
+<eagle version="6.6.0">
 <drawing>
 <settings>
@@
 <setting verticaltext="up"/>
 </settings>
-<grid distance="0.1" unitdist="inch" unit="inch" style="lines" multiple="1" display="no" altdistance="0.01" altunitdist="inch" altunit="inch"/>
+<grid distance="0.05" unitdist="inch" unit="inch" style="lines" multiple="1" display="no" altdistance="0.01" altunitdist="inch" altunit="inch"/>
 <layers>
 <layer number="1" name="Top" color="4" fill="1" visible="no" active="no"/>
@@
 <part name="J2" library="con-amp" deviceset="MTA08-100" device=""/>
 <part name="J3" library="con-amp" deviceset="MTA08-100" device=""/>
+<part name="P+3" library="supply1" deviceset="VCC" device=""/>
+<part name="P+4" library="supply1" deviceset="VCC" device=""/>
 </parts>
 <sheets>
@@
 <instance part="J2" gate="G$1" x="107.95" y="125.73" rot="MR270"/>
 <instance part="J3" gate="G$1" x="210.82" y="95.25" rot="R270"/>
+<instance part="P+3" gate="VCC" x="143.51" y="62.23"/>
+<instance part="P+4" gate="VCC" x="125.73" y="138.43"/>
 </instances>
 <busses>
@@
 </segment>
 </net>
-<net name="VCC" class="0">
+<net name="VDD_3.3V" class="0">
+<segment>
+<pinref part="P+2" gate="VCC" pin="VCC"/>
+<wire x1="196.85" y1="109.22" x2="196.85" y2="95.25" width="0.1524" layer="91"/>
+<wire x1="196.85" y1="95.25" x2="186.69" y2="95.25" width="0.1524" layer="91"/>
+<pinref part="J1" gate="G$1" pin="VDD_3.3V"/>
+</segment>
+<segment>
+<pinref part="J1" gate="G$1" pin="VDD_BATT"/>
+<wire x1="161.29" y1="64.77" x2="161.29" y2="57.15" width="0.1524" layer="91"/>
+<pinref part="P+3" gate="VCC" pin="VCC"/>
+<wire x1="161.29" y1="57.15" x2="143.51" y2="57.15" width="0.1524" layer="91"/>
+<wire x1="143.51" y1="57.15" x2="143.51" y2="59.69" width="0.1524" layer="91"/>
+</segment>
 <segment>
 <pinref part="XB1" gate="G$1" pin="VCC"/>
@@
 <wire x1="62.23" y1="106.68" x2="62.23" y2="113.03" width="0.1524" layer="91"/>
 </segment>
-</net>
-<net name="VDD_3.3V" class="0">
-<segment>
-<pinref part="P+2" gate="VCC" pin="VCC"/>
-<wire x1="196.85" y1="109.22" x2="196.85" y2="95.25" width="0.1524" layer="91"/>
-<wire x1="196.85" y1="95.25" x2="186.69" y2="95.25" width="0.1524" layer="91"/>
-<pinref part="J1" gate="G$1" pin="VDD_3.3V"/>
-</segment>
-</net>
+<segment>
+<pinref part="J1" gate="G$1" pin="VDD_3.3V_RF"/>
+<pinref part="P+4" gate="VCC" pin="VCC"/>
+<wire x1="128.27" y1="105.41" x2="125.73" y2="105.41" width="0.1524" layer="91"/>
+<wire x1="125.73" y1="105.41" x2="125.73" y2="135.89" width="0.1524" layer="91"/>
+</segment>
+</net>
